File: hardware/bus_board/bus_board.kicad_pcb (KiCad board)
At the start: 2 copper layers, 100 x 30 mm, 14 parts, among them J1 Eurorack Power, J2 Eurorack Power, J3 Eurorack Power, J4 Eurorack Power, J5 Eurorack Power, J6 Eurorack Power, J7 Eurorack Power

Commit message: Move some silkscreen around just a little
Parts:
- removed POLARITY: Symbol_Barrel_Polarity, Symbol:Symbol_Barrel_Polarity
Changed lines of the file:
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@@
     )
-  )
-  (footprint "Symbol:Symbol_Barrel_Polarity" (layer "F.Cu")
-    (at 119.2 105.975)
-    (descr "Barrel connector polarity indicator")
-    (tags "barrel polarity")
-    (attr board_only exclude_from_pos_files exclude_from_bom)
-    (fp_text reference "POLARITY" (at 0 -2) (layer "F.SilkS") hide
-      (effects (font (size 1 1) (thickness 0.15)))
-    )
-    (fp_text value "Symbol_Barrel_Polarity" (at 0 2) (layer "F.Fab")
-      (effects (font (size 1 1) (thickness 0.15)))
-    )
-    (fp_line (start 3.02 0.475) (end 3.02 -0.325) (layer "F.SilkS") (width 0.2))
-    (fp_line (start -2 0.075) (end -1.1 0.075) (layer "F.SilkS") (width 0.15))
-    (fp_line (start -3.41 0.08) (end -2.61 0.08) (layer "F.SilkS") (width 0.2))
-    (fp_line (start 0 0.075) (end 2 0.075) (layer "F.SilkS") (width 0.15))
-    (fp_line (start 2.62 0.075) (end 3.42 0.075) (layer "F.SilkS") (width 0.2))
-    (fp_arc (start 0.75 0.75) (mid -1.007627 0.128033) (end 0.675 -0.675) (layer "F.SilkS") (width 0.15))
-    (fp_circle (center -3 0.075) (end -3 1) (layer "F.SilkS") (width 0.15) (fill none))
-    (fp_circle (center 3 0.075) (end 3 1) (layer "F.SilkS") (width 0.15) (fill none))
-    (fp_circle (center 0 0.075) (end 0 0.25) (layer "F.SilkS") (width 0.5) (fill none))
   )
   (footprint "winterbloom:Eurorack_Power_2x8_Shrouded_Lock" (layer "F.Cu")

Commit message: Update the busboard with new name
Parts:
- removed G***: LOGO, LOGO
Other:
- board text added: "${COMMENT2} ${COMMENT3}"
- board text added: "${TITLE} ${REVISION} ${ISSUE_DATE}"
- board text removed: "${TITLE} ${REVISION} ${ISSUE_DATE} ${COMMENT2} ${COMMENT3}"

Commit message: Widen some traces- again
Changed lines of the file:
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@@
   (via (at 130.5 122.075) (size 0.7) (drill 0.3) (layers "F.Cu" "B.Cu") (free) (net 1))
   (via (at 125.5 122.075) (size 0.7) (drill 0.3) (layers "F.Cu" "B.Cu") (free) (net 1))
-  (segment (start 143.8141 106.805) (end 119.5146 106.805) (width 1) (layer "F.Cu") (net 2))
-  (segment (start 119.5146 106.805) (end 70.9156 106.805) (width 1) (layer "F.Cu") (net 2))
-  (segment (start 146.3541 106.805) (end 143.8141 106.805) (width 1) (layer "F.Cu") (net 2))
-  (segment (start 131.66435 116.965) (end 70.9156 116.965) (width 1) (layer "F.Cu") (net 3))
-  (segment (start 146.3541 116.965) (end 143.8141 116.965) (width 1) (layer "F.Cu") (net 3))
-  (segment (start 143.8141 116.965) (end 131.66435 116.965) (width 1) (layer "F.Cu") (net 3))
-  (segment (start 70.7124 104.265) (end 73.2524 104.265) (width 1) (layer "F.Cu") (net 4))
-  (segment (start 73.2524 104.265) (end 146.1509 104.265) (width 1) (layer "F.Cu") (net 4))
-  (segment (start 70.9156 101.725) (end 143.8141 101.725) (width 0.4) (layer "F.Cu") (net 5))
-  (segment (start 143.8141 101.725) (end 146.3541 101.725) (width 0.4) (layer "F.Cu") (net 5))
-  (segment (start 70.7124 99.185) (end 143.6109 99.185) (width 0.4) (layer "F.Cu") (net 6))
-  (segment (start 143.6109 99.185) (end 146.1509 99.185) (width 0.4) (layer "F.Cu") (net 6))
+  (segment (start 70.9156 106.805) (end 146.3541 106.805) (width 1.5) (layer "F.Cu") (net 2))
+  (segment (start 70.9156 116.965) (end 146.3541 116.965) (width 1.5) (layer "F.Cu") (net 3))
+  (segment (start 70.7124 104.265) (end 146.1509 104.265) (width 1.5) (layer "F.Cu") (net 4))
+  (segment (start 70.9156 101.725) (end 146.3541 101.725) (width 0.8) (layer "F.Cu") (net 5))
+  (segment (start 146.1509 99.185) (end 70.7124 99.185) (width 0.8) (layer "F.Cu") (net 6))
   (zone (net 1) (net_name "GND") (layer "F.Cu") (hatch edge 0.508)
     (connect_pads thru_hole_only (clearance 0.254))

Commit message: hardware: use fancytext labels on busboard
Parts:
- added G***: LOGO, LOGO, F.Cu at (63.0, 114.9)
- added G***: LOGO, LOGO, F.Cu at (153.7, 115.0)
Other:
- board text removed: "RED STRIPE"
