File: hardware/bus_board/bus_board.kicad_sch (KiCad schematic)
At the start: 11 parts, among them J1 Eurorack Power, J2 Eurorack Power, J3 Eurorack Power, J4 Eurorack Power, J5 Eurorack Power, J6 Eurorack Power, J7 Eurorack Power

Commit message: Update the busboard with new name
Other:
- title: Nickel: bus board -> Micronova bus board
Changed lines of the file:
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@@
   (paper "USLetter")
   (title_block
-    (title "Nickel: bus board")
-    (date "2022-06-13")
-    (rev "v1")
+    (title "Micronova bus board")
+    (date "2022-07-31")
+    (rev "v2")
     (company "Winterbloom")
     (comment 1 "Alethea Flowers")
     (comment 2 "CERN-OHL-P V2")
+    (comment 3 "micronova.wntr.dev")
   )
   (junction (at 139.065 194.945) (diameter 0) (color 0 0 0 0)
