File: hardware/board/board.kicad_sch (KiCad schematic)
At the start: 38 parts, among them J1 DC THRU, J2 DC THRU, J3 DC OUT, J4 DC IN, J5 DC IN, J6 DC OUT, J7 Eurorack Power, J8 Eurorack Power, SW1 ON/OFF, U1 VX7805-500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

Commit message: Update page details in schematic
Other:
- company: (none) -> Winterbloom
- title: (none) -> Nickel
Changed lines of the file:
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@@
   (paper "USLetter")
   (title_block
-    (date "2022-05-10")
+    (title "Nickel")
+    (date "2022-05-23")
+    (rev "v2")
+    (company "Winterbloom")
+    (comment 1 "Alethea Flowers")
+    (comment 2 "CERN-OHL-P V2")
   )
   (junction (at 139.065 194.945) (diameter 0) (color 0 0 0 0)

Commit message: Use new winterbloom footprints
Parts:
- J2, J3, J4, J6, SW1: footprint winterbloom:TerminalBlock_4Ucon_1x02_P3.50mm_Horizontal -> winterbloom:TerminalBlock_4UCON_1x02_P3.50mm_Horizontal
- J7, J8: footprint winterbloom:IDC-Header_2x08_P2.54mm_Vertical_Press_Fit -> winterbloom:Eurorack_Power_2x8_Shrouded_Lock
- U1: footprint winterbloom:CUI_VX78 -> winterbloom:Converter_DCDC_CUI_VX78-500_THT
- U2, U3: footprint winterbloom:CUI_P78E -> winterbloom:Converter_DCDC_CUI_P78E-1000_THT
Changed lines of the file:
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@@
     (property "Reference" "SW1" (id 0) (at 44.45 83.82 0))
     (property "Value" "ON/OFF" (id 1) (at 44.45 86.36 0))
-    (property "Footprint" "winterbloom:TerminalBlock_4Ucon_1x02_P3.50mm_Horizontal" (id 2) (at 44.45 90.17 0)
+    (property "Footprint" "winterbloom:TerminalBlock_4UCON_1x02_P3.50mm_Horizontal" (id 2) (at 44.45 90.17 0)
       (effects (font (size 1.27 1.27)) hide)
     )
@@
     (property "Reference" "U1" (id 0) (at 147.955 45.881 0))
     (property "Value" "VX7805-500" (id 1) (at 147.955 48.4179 0))
-    (property "Footprint" "winterbloom:CUI_VX78" (id 2) (at 147.955 54.61 0)
+    (property "Footprint" "winterbloom:Converter_DCDC_CUI_VX78-500_THT" (id 2) (at 147.955 54.61 0)
       (effects (font (size 1.27 1.27)) hide)
     )
@@
     (property "Reference" "U2" (id 0) (at 147.955 81.441 0))
     (property "Value" "P78E-1000" (id 1) (at 147.955 83.9779 0))
-    (property "Footprint" "winterbloom:CUI_P78E" (id 2) (at 147.955 90.17 0)
+    (property "Footprint" "winterbloom:Converter_DCDC_CUI_P78E-1000_THT" (id 2) (at 147.955 90.17 0)
       (effects (font (size 1.27 1.27)) hide)
     )
@@
     (property "Reference" "J6" (id 0) (at 241.935 35.0352 0))
     (property "Value" "DC OUT" (id 1) (at 241.935 37.5721 0))
-    (property "Footprint" "winterbloom:TerminalBlock_4Ucon_1x02_P3.50mm_Horizontal" (id 2) (at 241.935 40.005 0)
+    (property "Footprint" "winterbloom:TerminalBlock_4UCON_1x02_P3.50mm_Horizontal" (id 2) (at 241.935 40.005 0)
       (effects (font (size 1.27 1.27)) hide)
     )
@@
     (property "Reference" "J8" (id 0) (at 246.38 59.1652 0))
     (property "Value" "Eurorack Power" (id 1) (at 246.38 61.7021 0))
-    (property "Footprint" "winterbloom:IDC-Header_2x08_P2.54mm_Vertical_Press_Fit" (id 2) (at 245.11 71.755 0)
+    (property "Footprint" "winterbloom:Eurorack_Power_2x8_Shrouded_Lock" (id 2) (at 245.11 71.755 0)
       (effects (font (size 1.27 1.27)) hide)
     )
@@
     (property "Reference" "J4" (id 0) (at 56.515 18.5252 0))
     (property "Value" "DC IN" (id 1) (at 56.515 21.0621 0))
-    (property "Footprint" "winterbloom:TerminalBlock_4Ucon_1x02_P3.50mm_Horizontal" (id 2) (at 56.515 23.495 0)
+    (property "Footprint" "winterbloom:TerminalBlock_4UCON_1x02_P3.50mm_Horizontal" (id 2) (at 56.515 23.495 0)
       (effects (font (size 1.27 1.27)) hide)
     )
@@
     (property "Reference" "J3" (id 0) (at 241.935 19.7952 0))
     (property "Value" "DC OUT" (id 1) (at 241.935 22.3321 0))
-    (property "Footprint" "winterbloom:TerminalBlock_4Ucon_1x02_P3.50mm_Horizontal" (id 2) (at 241.935 24.765 0)
+    (property "Footprint" "winterbloom:TerminalBlock_4UCON_1x02_P3.50mm_Horizontal" (id 2) (at 241.935 24.765 0)
       (effects (font (size 1.27 1.27)) hide)
     )
@@
     (property "Reference" "J2" (id 0) (at 56.515 35.0352 0))
     (property "Value" "DC THRU" (id 1) (at 56.515 37.5721 0))
-    (property "Footprint" "winterbloom:TerminalBlock_4Ucon_1x02_P3.50mm_Horizontal" (id 2) (at 56.515 40.005 0)
+    (property "Footprint" "winterbloom:TerminalBlock_4UCON_1x02_P3.50mm_Horizontal" (id 2) (at 56.515 40.005 0)
       (effects (font (size 1.27 1.27)) hide)
     )
@@
     (property "Reference" "U3" (id 0) (at 147.955 112.556 0))
     (property "Value" "P78E-1000" (id 1) (at 147.955 115.0929 0))
-    (property "Footprint" "winterbloom:CUI_P78E" (id 2) (at 147.955 121.285 0)
+    (property "Footprint" "winterbloom:Converter_DCDC_CUI_P78E-1000_THT" (id 2) (at 147.955 121.285 0)
       (effects (font (size 1.27 1.27)) hide)
     )
@@
     (property "Reference" "J7" (id 0) (at 246.38 95.3602 0))
     (property "Value" "Eurorack Power" (id 1) (at 246.38 97.8971 0))
-    (property "Footprint" "winterbloom:IDC-Header_2x08_P2.54mm_Vertical_Press_Fit" (id 2) (at 245.11 107.95 0)
+    (property "Footprint" "winterbloom:Eurorack_Power_2x8_Shrouded_Lock" (id 2) (at 245.11 107.95 0)
       (effects (font (size 1.27 1.27)) hide)
     )
@@
     )
     (path "/9bb0dca3-93e9-4fb8-8df7-0a69ab0c8d6b"
-      (reference "J2") (unit 1) (value "DC THRU") (footprint "winterbloom:TerminalBlock_4Ucon_1x02_P3.50mm_Horizontal")
+      (reference "J2") (unit 1) (value "DC THRU") (footprint "winterbloom:TerminalBlock_4UCON_1x02_P3.50mm_Horizontal")
     )
     (path "/983728d1-7fc3-4e3b-9bf7-f751ee104cc1"
-      (reference "J3") (unit 1) (value "DC OUT") (footprint "winterbloom:TerminalBlock_4Ucon_1x02_P3.50mm_Horizontal")
+      (reference "J3") (unit 1) (value "DC OUT") (footprint "winterbloom:TerminalBlock_4UCON_1x02_P3.50mm_Horizontal")
     )
     (path "/3f19a83e-b299-4289-8ee0-190dd22509bf"
-      (reference "J4") (unit 1) (value "DC IN") (footprint "winterbloom:TerminalBlock_4Ucon_1x02_P3.50mm_Horizontal")
+      (reference "J4") (unit 1) (value "DC IN") (footprint "winterbloom:TerminalBlock_4UCON_1x02_P3.50mm_Horizontal")
     )
     (path "/a7c6f048-0ad7-4885-bb19-538c9404fc2a"
@@
     )
     (path "/24dbae12-9d1d-425e-b5d7-18a8685dd80d"
-      (reference "J6") (unit 1) (value "DC OUT") (footprint "winterbloom:TerminalBlock_4Ucon_1x02_P3.50mm_Horizontal")
+      (reference "J6") (unit 1) (value "DC OUT") (footprint "winterbloom:TerminalBlock_4UCON_1x02_P3.50mm_Horizontal")
     )
     (path "/fa0dbe8b-75a2-4a32-9d90-1f26c2f28af8"
-      (reference "J7") (unit 1) (value "Eurorack Power") (footprint "winterbloom:IDC-Header_2x08_P2.54mm_Vertical_Press_Fit")
+      (reference "J7") (unit 1) (value "Eurorack Power") (footprint "winterbloom:Eurorack_Power_2x8_Shrouded_Lock")
     )
     (path "/3d1d0df1-55e0-40ad-a6af-e205879cb36e"
-      (reference "J8") (unit 1) (value "Eurorack Power") (footprint "winterbloom:IDC-Header_2x08_P2.54mm_Vertical_Press_Fit")
+      (reference "J8") (unit 1) (value "Eurorack Power") (footprint "winterbloom:Eurorack_Power_2x8_Shrouded_Lock")
     )
     (path "/185a4d14-ba2c-4702-bd00-0c5a75f6b32e"
@@
     )
     (path "/05cdb9b6-c0dc-4fe6-92b4-e0c4062a70ca"
-      (reference "SW1") (unit 1) (value "ON/OFF") (footprint "winterbloom:TerminalBlock_4Ucon_1x02_P3.50mm_Horizontal")
+      (reference "SW1") (unit 1) (value "ON/OFF") (footprint "winterbloom:TerminalBlock_4UCON_1x02_P3.50mm_Horizontal")
     )
     (path "/55f2b110-ae00-4e29-87a8-6e03ae68c4a4"
@@
     )
     (path "/192bf8fd-d307-4fe5-ad18-c9ef0bed1880"
-      (reference "U1") (unit 1) (value "VX7805-500") (footprint "winterbloom:CUI_VX78")
+      (reference "U1") (unit 1) (value "VX7805-500") (footprint "winterbloom:Converter_DCDC_CUI_VX78-500_THT")
     )
     (path "/22836a84-b49b-4545-bc98-bc59bbc21932"
-      (reference "U2") (unit 1) (value "P78E-1000") (footprint "winterbloom:CUI_P78E")
+      (reference "U2") (unit 1) (value "P78E-1000") (footprint "winterbloom:Converter_DCDC_CUI_P78E-1000_THT")
     )
     (path "/c5dbc2f4-347d-4e8b-9dc5-05ae6c8ee4e9"
-      (reference "U3") (unit 1) (value "P78E-1000") (footprint "winterbloom:CUI_P78E")
-    )
-  )
+      (reference "U3") (unit 1) (value "P78E-1000") (footprint "winterbloom:Converter_DCDC_CUI_P78E-1000_THT")
+    )
+  )
